Commit message: add ridgeback desc; correct ur5_robot macro call; working

File: ridgeback_ur5_description/urdf/ridgeback_ur5_description.urdf.xacro (robot description, xacro)
@@ -1,5 +1,17 @@
-<?xml version="1.0"?>
-<robot xmlns:xacro="http://ros.org/wiki/xacro">
-  <xacro:include filename="$(find ur_description)/urdf/inc/ur5_macro.xacro" />
+<robot xmlns:xacro="http://ros.org/wiki/xacro" name="ridgeback_ur5">
+  <xacro:arg name="ur_type" default="ur5"/>
+  <xacro:include filename="$(find ur_description)/urdf/ur_macro.xacro" />
+  <xacro:include filename="$(find ridgeback_description)/urdf/ridgeback.urdf.xacro" />
+  <xacro:ur_robot
+    name="ur5"
+    ur_type="$(arg ur_type)"
+    tf_prefix="ur_arm_"
+    parent="mid_mount"
+    joint_limits_parameters_file="$(find ur_description)/config/$(arg ur_type)/joint_limits.yaml"
+    kinematics_parameters_file="$(find ur_description)/config/$(arg ur_type)/default_kinematics.yaml"
+    physical_parameters_file="$(find ur_description)/config/$(arg ur_type)/physical_parameters.yaml"
+    visual_parameters_file="$(find ur_description)/config/$(arg ur_type)/visual_parameters.yaml">
+    <origin xyz="0 0 0" rpy="0 0 0" />
+  </xacro:ur_robot>
   <joint name="arm_mount_joint" type="fixed">
     <parent link="mid_mount" />
@@ -7,4 +19,4 @@
     <origin xyz="$(optenv RIDGEBACK_UR_XYZ 0 0 0)" rpy="$(optenv RIDGEBACK_UR_RPY 0 0 0)"/>
   </joint>
-  <xacro:ur5_robot prefix="ur_arm_" />
+  <!-- <link name="world"/> -->
 </robot>

Commit message: include call to ur_robot macro

File: ridgeback_ur5_description/urdf/ridgeback_ur5_description.urdf.xacro (robot description, xacro)
@@ -1,23 +1,63 @@
 <?xml version="1.0"?>
 <robot xmlns:xacro="http://ros.org/wiki/xacro" name="ridgeback_ur5">
+  <xacro:arg name="name" default="ur5"/>
   <xacro:arg name="ur_type" default="ur5"/>
-  <xacro:include filename="$(find ur_description)/urdf/ur_macro.xacro" />
-  <xacro:include filename="$(find ridgeback_description)/urdf/ridgeback.urdf.xacro" />
-  <xacro:ur_robot
-    name="ur5"
+  <xacro:arg name="sim_ignition" default="true"/>
+  <xacro:arg name="tf_prefix" default="ur_arm_" />
+  <xacro:arg name="parent" default="mid_mount" /> <!--world-->
+  <xacro:arg name="joint_limit_params" default="$(find ur_description)/config/$(arg ur_type)/joint_limits.yaml"/>
+  <xacro:arg name="kinematics_params" default="$(find ur_description)/config/$(arg ur_type)/default_kinematics.yaml"/>
+  <xacro:arg name="physical_params" default="$(find ur_description)/config/$(arg ur_type)/physical_parameters.yaml"/>
+  <xacro:arg name="visual_params" default="$(find ur_description)/config/$(arg ur_type)/visual_parameters.yaml"/>
+  <xacro:arg name="transmission_hw_interface" default="hardware_interface/PositionJointInterface"/>
+  <xacro:arg name="use_fake_hardware" default="false" />
+  <xacro:arg name="fake_sensor_commands" default="false" />
+  <xacro:arg name="sim_gazebo" default="false" />
+  <xacro:arg name="sim_ignition" default="true" />
+  <xacro:arg name="headless_mode" default="false" />
+  <!-- initial position for simulations (Fake Hardware, Gazebo, Ignition) -->
+  <xacro:arg name="initial_positions_file" default="$(find ur_description)/config/initial_positions.yaml"/>
+  <!-- convert to property to use substitution in function -->
+  <xacro:property name="initial_positions_file" default="$(arg initial_positions_file)"/>
+  <!-- <xacro:ur_robot
+    name="$(arg name)"
     ur_type="$(arg ur_type)"
     tf_prefix="ur_arm_"
-    parent="mid_mount"
+    parent="world"
     joint_limits_parameters_file="$(find ur_description)/config/$(arg ur_type)/joint_limits.yaml"
     kinematics_parameters_file="$(find ur_description)/config/$(arg ur_type)/default_kinematics.yaml"
     physical_parameters_file="$(find ur_description)/config/$(arg ur_type)/physical_parameters.yaml"
-    visual_parameters_file="$(find ur_description)/config/$(arg ur_type)/visual_parameters.yaml">
-    <origin xyz="0 0 0" rpy="0 0 0" />
+    visual_parameters_file="$(find ur_description)/config/$(arg ur_type)/visual_parameters.yaml"
+    sim_ignition="$(arg sim_ignition)">
+    <origin xyz="$(optenv RIDGEBACK_UR_XYZ 0 0 0)" rpy="$(optenv RIDGEBACK_UR_RPY 0 0 0)"/>
+  </xacro:ur_robot> -->
+  <!-- arm -->
+  <xacro:ur_robot
+    name="$(arg name)"
+    ur_type="$(arg ur_type)"
+    tf_prefix="$(arg tf_prefix)"
+    parent="$(arg parent)"
+    joint_limits_parameters_file="$(arg joint_limit_params)"
+    kinematics_parameters_file="$(arg kinematics_params)"
+    physical_parameters_file="$(arg physical_params)"
+    visual_parameters_file="$(arg visual_params)"
+    transmission_hw_interface="$(arg transmission_hw_interface)"
+    use_fake_hardware="$(arg use_fake_hardware)"
+    fake_sensor_commands="$(arg fake_sensor_commands)"
+    sim_gazebo="$(arg sim_gazebo)"
+    sim_ignition="$(arg sim_ignition)"
+    headless_mode="$(arg headless_mode)"
+    initial_positions="${xacro.load_yaml(initial_positions_file)}"
+    >
+    <!-- position robot in the world -->
+    <origin xyz="$(optenv RIDGEBACK_UR_XYZ 0 0 0)" rpy="$(optenv RIDGEBACK_UR_RPY 0 0 0)"/>
   </xacro:ur_robot>
-  <joint name="arm_mount_joint" type="fixed">
+  <!-- <joint name="arm_mount_joint" type="fixed">
     <parent link="mid_mount" />
     <child link="ur_arm_base_link" />
     <origin xyz="$(optenv RIDGEBACK_UR_XYZ 0 0 0)" rpy="$(optenv RIDGEBACK_UR_RPY 0 0 0)"/>
-  </joint>
-  <!-- <link name="world"/> -->
+  </joint> -->
+  <!-- <link name="world"/>  -->
+  <xacro:include filename="$(find ur_description)/urdf/ur.urdf.xacro" />
+  <xacro:include filename="$(find ridgeback_description)/urdf/ridgeback.urdf.xacro" />
 </robot>

Commit message: include ur5_robotiq_85_gripper urdf

File: ridgeback_ur5_description/urdf/ridgeback_ur5_description.urdf.xacro (robot description, xacro)
@@ -5,9 +5,9 @@
   <xacro:arg name="sim_ignition" default="true"/>
   <xacro:arg name="tf_prefix" default="ur_arm_" />
-  <xacro:arg name="parent" default="mid_mount" /> <!--world-->
-  <xacro:arg name="joint_limit_params" default="$(find ur_description)/config/$(arg ur_type)/joint_limits.yaml"/>
-  <xacro:arg name="kinematics_params" default="$(find ur_description)/config/$(arg ur_type)/default_kinematics.yaml"/>
-  <xacro:arg name="physical_params" default="$(find ur_description)/config/$(arg ur_type)/physical_parameters.yaml"/>
-  <xacro:arg name="visual_params" default="$(find ur_description)/config/$(arg ur_type)/visual_parameters.yaml"/>
+  <xacro:arg name="parent" default="world" /> <!--mid_mount-->
+  <xacro:arg name="joint_limit_params" default="$(find ur5_robotiq_description)/config/$(arg ur_type)/joint_limits.yaml"/>
+  <xacro:arg name="kinematics_params" default="$(find ur5_robotiq_description)/config/$(arg ur_type)/default_kinematics.yaml"/>
+  <xacro:arg name="physical_params" default="$(find ur5_robotiq_description)/config/$(arg ur_type)/physical_parameters.yaml"/>
+  <xacro:arg name="visual_params" default="$(find ur5_robotiq_description)/config/$(arg ur_type)/visual_parameters.yaml"/>
   <xacro:arg name="transmission_hw_interface" default="hardware_interface/PositionJointInterface"/>
   <xacro:arg name="use_fake_hardware" default="false" />
@@ -17,7 +17,9 @@
   <xacro:arg name="headless_mode" default="false" />
   <!-- initial position for simulations (Fake Hardware, Gazebo, Ignition) -->
-  <xacro:arg name="initial_positions_file" default="$(find ur_description)/config/initial_positions.yaml"/>
+  <xacro:arg name="initial_positions_file" default="$(find ur5_robotiq_description)/config/$(arg ur_type)/initial_positions.yaml"/>
   <!-- convert to property to use substitution in function -->
   <xacro:property name="initial_positions_file" default="$(arg initial_positions_file)"/>
+  <!-- <xacro:include filename="$(find ur5_robotiq_description)/urdf/ur.urdf.xacro" /> -->
+  <!-- <xacro:include filename="$(find ridgeback_description)/urdf/ridgeback.urdf.xacro" /> -->
   <!-- <xacro:ur_robot
     name="$(arg name)"
@@ -25,11 +27,12 @@
     tf_prefix="ur_arm_"
     parent="world"
-    joint_limits_parameters_file="$(find ur_description)/config/$(arg ur_type)/joint_limits.yaml"
-    kinematics_parameters_file="$(find ur_description)/config/$(arg ur_type)/default_kinematics.yaml"
-    physical_parameters_file="$(find ur_description)/config/$(arg ur_type)/physical_parameters.yaml"
-    visual_parameters_file="$(find ur_description)/config/$(arg ur_type)/visual_parameters.yaml"
+    joint_limits_parameters_file="$(find ur5_robotiq_description)/config/$(arg ur_type)/joint_limits.yaml"
+    kinematics_parameters_file="$(find ur5_robotiq_description)/config/$(arg ur_type)/default_kinematics.yaml"
+    physical_parameters_file="$(find ur5_robotiq_description)/config/$(arg ur_type)/physical_parameters.yaml"
+    visual_parameters_file="$(find ur5_robotiq_description)/config/$(arg ur_type)/visual_parameters.yaml"
     sim_ignition="$(arg sim_ignition)">
     <origin xyz="$(optenv RIDGEBACK_UR_XYZ 0 0 0)" rpy="$(optenv RIDGEBACK_UR_RPY 0 0 0)"/>
   </xacro:ur_robot> -->
+  <xacro:include filename="$(find ur5_robotiq_description)/urdf/ur5_robotiq_85_gripper.urdf.xacro" />
   <!-- arm -->
   <xacro:ur_robot
@@ -58,6 +61,4 @@
     <origin xyz="$(optenv RIDGEBACK_UR_XYZ 0 0 0)" rpy="$(optenv RIDGEBACK_UR_RPY 0 0 0)"/>
   </joint> -->
-  <!-- <link name="world"/>  -->
-  <xacro:include filename="$(find ur_description)/urdf/ur.urdf.xacro" />
-  <xacro:include filename="$(find ridgeback_description)/urdf/ridgeback.urdf.xacro" />
+  <link name="world"/>
 </robot>
