Commit message: package://->file://; add robotiq_gripper_ros2_control macro

File: ur5_robotiq_description/urdf/robotiq_85/robotiq_85_gripper.urdf.xacro (robot description, xacro)
@@ -1,6 +1,9 @@
 <?xml version="1.0"?>
 <robot name="robotiq_85_gripper" xmlns:xacro="http://www.ros.org/wiki/xacro">
-  <xacro:include filename="$(find ur5_robotiq_description)/urdf/robotiq_85/robotiq_85_gripper.transmission.xacro" />
+  <!-- <xacro:include filename="$(find ur5_robotiq_description)/urdf/robotiq_85/robotiq_85_gripper.transmission.xacro" /> -->
   <xacro:macro name="robotiq_85_gripper" params="prefix parent *origin">
+    <!-- ros2 control include -->
+    <xacro:include filename="$(find ur5_robotiq_description)/urdf/robotiq_85/robotiq_85.ros2_control.xacro" />
+    <xacro:robotiq_gripper_ros2_control prefix="${prefix}"/>
     <joint name="${prefix}robotiq_85_base_joint" type="fixed">
       <parent link="${parent}"/>
@@ -11,10 +14,10 @@
       <visual>
         <geometry>
-          <mesh filename="package://ur5_robotiq_description/meshes/robotiq_85/visual/robotiq_85_base_link.dae"/>
-        </geometry>
-      </visual>
-      <collision>
-        <geometry>
-          <mesh filename="package://ur5_robotiq_description/meshes/robotiq_85/collision/robotiq_85_base_link.stl"/>
+          <mesh filename="file://ur5_robotiq_description/meshes/robotiq_85/visual/robotiq_85_base_link.dae"/>
+        </geometry>
+      </visual>
+      <collision>
+        <geometry>
+          <mesh filename="file://ur5_robotiq_description/meshes/robotiq_85/collision/robotiq_85_base_link.stl"/>
         </geometry>
       </collision>
@@ -45,10 +48,10 @@
       <visual>
         <geometry>
-          <mesh filename="package://ur5_robotiq_description/meshes/robotiq_85/visual/robotiq_85_knuckle_link.dae"/>
-        </geometry>
-      </visual>
-      <collision>
-        <geometry>
-          <mesh filename="package://ur5_robotiq_description/meshes/robotiq_85/collision/robotiq_85_knuckle_link.stl"/>
+          <mesh filename="file://ur5_robotiq_description/meshes/robotiq_85/visual/robotiq_85_knuckle_link.dae"/>
+        </geometry>
+      </visual>
+      <collision>
+        <geometry>
+          <mesh filename="file://ur5_robotiq_description/meshes/robotiq_85/collision/robotiq_85_knuckle_link.stl"/>
         </geometry>
       </collision>
@@ -64,10 +67,10 @@
       <visual>
         <geometry>
-          <mesh filename="package://ur5_robotiq_description/meshes/robotiq_85/visual/robotiq_85_knuckle_link.dae"/>
-        </geometry>
-      </visual>
-      <collision>
-        <geometry>
-          <mesh filename="package://ur5_robotiq_description/meshes/robotiq_85/collision/robotiq_85_knuckle_link.stl"/>
+          <mesh filename="file://ur5_robotiq_description/meshes/robotiq_85/visual/robotiq_85_knuckle_link.dae"/>
+        </geometry>
+      </visual>
+      <collision>
+        <geometry>
+          <mesh filename="file://ur5_robotiq_description/meshes/robotiq_85/collision/robotiq_85_knuckle_link.stl"/>
         </geometry>
       </collision>
@@ -93,10 +96,10 @@
       <visual>
         <geometry>
-          <mesh filename="package://ur5_robotiq_description/meshes/robotiq_85/visual/robotiq_85_finger_link.dae"/>
-        </geometry>
-      </visual>
-      <collision>
-        <geometry>
-          <mesh filename="package://ur5_robotiq_description/meshes/robotiq_85/collision/robotiq_85_finger_link.stl"/>
+          <mesh filename="file://ur5_robotiq_description/meshes/robotiq_85/visual/robotiq_85_finger_link.dae"/>
+        </geometry>
+      </visual>
+      <collision>
+        <geometry>
+          <mesh filename="file://ur5_robotiq_description/meshes/robotiq_85/collision/robotiq_85_finger_link.stl"/>
         </geometry>
       </collision>
@@ -112,10 +115,10 @@
       <visual>
         <geometry>
-          <mesh filename="package://ur5_robotiq_description/meshes/robotiq_85/visual/robotiq_85_finger_link.dae"/>
-        </geometry>
-      </visual>
-      <collision>
-        <geometry>
-          <mesh filename="package://ur5_robotiq_description/meshes/robotiq_85/collision/robotiq_85_finger_link.stl"/>
+          <mesh filename="file://ur5_robotiq_description/meshes/robotiq_85/visual/robotiq_85_finger_link.dae"/>
+        </geometry>
+      </visual>
+      <collision>
+        <geometry>
+          <mesh filename="file://ur5_robotiq_description/meshes/robotiq_85/collision/robotiq_85_finger_link.stl"/>
         </geometry>
       </collision>
@@ -147,10 +150,10 @@
       <visual>
         <geometry>
-          <mesh filename="package://ur5_robotiq_description/meshes/robotiq_85/visual/robotiq_85_inner_knuckle_link.dae"/>
-        </geometry>
-      </visual>
-      <collision>
-        <geometry>
-          <mesh filename="package://ur5_robotiq_description/meshes/robotiq_85/collision/robotiq_85_inner_knuckle_link.stl"/>
+          <mesh filename="file://ur5_robotiq_description/meshes/robotiq_85/visual/robotiq_85_inner_knuckle_link.dae"/>
+        </geometry>
+      </visual>
+      <collision>
+        <geometry>
+          <mesh filename="file://ur5_robotiq_description/meshes/robotiq_85/collision/robotiq_85_inner_knuckle_link.stl"/>
         </geometry>
       </collision>
@@ -166,10 +169,10 @@
       <visual>
         <geometry>
-          <mesh filename="package://ur5_robotiq_description/meshes/robotiq_85/visual/robotiq_85_inner_knuckle_link.dae"/>
-        </geometry>
-      </visual>
-      <collision>
-        <geometry>
-          <mesh filename="package://ur5_robotiq_description/meshes/robotiq_85/collision/robotiq_85_inner_knuckle_link.stl"/>
+          <mesh filename="file://ur5_robotiq_description/meshes/robotiq_85/visual/robotiq_85_inner_knuckle_link.dae"/>
+        </geometry>
+      </visual>
+      <collision>
+        <geometry>
+          <mesh filename="file://ur5_robotiq_description/meshes/robotiq_85/collision/robotiq_85_inner_knuckle_link.stl"/>
         </geometry>
       </collision>
@@ -201,10 +204,10 @@
       <visual>
         <geometry>
-          <mesh filename="package://ur5_robotiq_description/meshes/robotiq_85/visual/robotiq_85_finger_tip_link.dae"/>
-        </geometry>
-      </visual>
-      <collision>
-        <geometry>
-          <mesh filename="package://ur5_robotiq_description/meshes/robotiq_85/collision/robotiq_85_finger_tip_link.stl"/>
+          <mesh filename="file://ur5_robotiq_description/meshes/robotiq_85/visual/robotiq_85_finger_tip_link.dae"/>
+        </geometry>
+      </visual>
+      <collision>
+        <geometry>
+          <mesh filename="file://ur5_robotiq_description/meshes/robotiq_85/collision/robotiq_85_finger_tip_link.stl"/>
         </geometry>
       </collision>
@@ -220,10 +223,10 @@
       <visual>
         <geometry>
-          <mesh filename="package://ur5_robotiq_description/meshes/robotiq_85/visual/robotiq_85_finger_tip_link.dae"/>
-        </geometry>
-      </visual>
-      <collision>
-        <geometry>
-          <mesh filename="package://ur5_robotiq_description/meshes/robotiq_85/collision/robotiq_85_finger_tip_link.stl"/>
+          <mesh filename="file://ur5_robotiq_description/meshes/robotiq_85/visual/robotiq_85_finger_tip_link.dae"/>
+        </geometry>
+      </visual>
+      <collision>
+        <geometry>
+          <mesh filename="file://ur5_robotiq_description/meshes/robotiq_85/collision/robotiq_85_finger_tip_link.stl"/>
         </geometry>
       </collision>
@@ -237,5 +240,5 @@
     </link>
     <!-- Improve grasping physics -->
-    <gazebo reference="${prefix}robotiq_85_left_finger_tip_link">
+    <!-- <gazebo reference="${prefix}robotiq_85_left_finger_tip_link">
       <kp>1000000.0</kp>
       <kd>1.0</kd>
@@ -250,6 +253,6 @@
       <mu2>1.0</mu2>
       <minDepth>0.001</minDepth>
-    </gazebo>
-    <xacro:robotiq_85_gripper_transmission prefix="${prefix}" />
+    </gazebo> -->
+    <!-- <xacro:robotiq_85_gripper_transmission prefix="${prefix}" /> -->
   </xacro:macro>
 </robot>
