Commit message: comment out gazebo classic mimic plugin

File: ur5_robotiq_description/urdf/robotiq_85/robotiq_85_gripper.transmission.xacro (robot description, xacro)
@@ -5,15 +5,23 @@
       <type>transmission_interface/SimpleTransmission</type>
       <joint name="${prefix}robotiq_85_left_knuckle_joint">
+        <hardwareInterface>hardware_interface/PositionJointInterface</hardwareInterface>
+      </joint>
+      <actuator name="${prefix}robotiq_85_left_knuckle_motor">
+        <hardwareInterface>hardware_interface/PositionJointInterface</hardwareInterface>
+        <mechanicalReduction>1</mechanicalReduction>
+      </actuator>
+    </transmission>
+    <!-- <transmission name="${prefix}robotiq_85_left_knuckle_trans">
+      <type>transmission_interface/SimpleTransmission</type>
+      <joint name="${prefix}robotiq_85_left_knuckle_joint">
         <hardwareInterface>hardware_interface/EffortJointInterface</hardwareInterface>
-        <!-- <hardwareInterface>EffortJointInterface</hardwareInterface> -->
       </joint>
       <actuator name="${prefix}robotiq_85_left_knuckle_motor">
         <mechanicalReduction>1</mechanicalReduction>
         <hardwareInterface>hardware_interface/EffortJointInterface</hardwareInterface>
-        <!-- <hardwareInterface>EfforJointInterface</hardwareInterface> -->
       </actuator>
-    </transmission>
+    </transmission> -->
     <!-- Mimic joints -->
-    <gazebo>
+    <!-- <gazebo>
       <plugin filename="libgazebo_mimic_joint_plugin.so" name="${prefix}mimic_robotiq_85_1">
         <joint>${prefix}robotiq_85_left_knuckle_joint</joint>
@@ -40,5 +48,5 @@
         <offset>0.0</offset>
       </plugin>
-    </gazebo>
+    </gazebo> -->
   </xacro:macro>
 </robot>
